Commit message: had to change the urdf limits

File: src/sim_pkg/sim_pkg/assets/bracketbot_v1_rev1/robot_continuous.urdf (robot description, URDF)
Before this commit: robot bracketbot_v1_rev1, 4 links, 3 joints
Joints:
- joint drive_left: limit lower=-3.141592653589793 upper=3.141592653589793 effort=10 velocity=10 -> lower=-3.141592653589793 upper=3.141592653589793 effort=1000 velocity=400
- joint drive_right: limit lower=-3.141592653589793 upper=3.141592653589793 effort=10 velocity=10 -> lower=-3.141592653589793 upper=3.141592653589793 effort=1000 velocity=400
